File: led-pcb.kicad_pcb (KiCad board)
At the start: 2 copper layers, 142 parts, among them IC1 HT16K33A-28SSOP, J1 Conn_01x04_Pin

Commit message: e
Parts:
- R1, R2, R3, R4, R5, R6, R7, R8: footprint Resistor_SMD:R_0603_1608Metric -> Resistor_SMD:R_0603_1608Metric_Pad0.98x0.95mm_HandSolder
- moved R8 69.8 mm to (99.0, 122.0)
- moved R7 69.5 mm to (99.0, 119.0)
- moved R6 69.2 mm to (99.0, 116.0)
- moved R5 68.9 mm to (99.0, 113.0)
- moved R4 68.6 mm to (99.0, 110.0)
- moved R3 68.3 mm to (99.0, 107.0)
- moved R2 68.0 mm to (99.0, 104.0)
- moved R1 67.7 mm to (99.0, 101.0)
- moved J1 60.5 mm to (185.0, 114.0)
- moved D8 46.4 mm to (104.0, 122.0)
- moved D7 46.0 mm to (104.0, 119.0)
- moved D120 45.9 mm to (160.0, 122.0)
- moved D6 45.6 mm to (104.0, 116.0)
- moved D119 45.5 mm to (160.0, 119.0)
- moved D24 45.5 mm to (112.0, 122.0)
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Connections:
- C2 pad 1: Net-(IC1-VSS) -> Net-(J1-Pin_2)
- C2 pad 2: Net-(J1-Pin_2) -> Net-(IC1-VSS)
Routing:
- net row0: track 0.00 -> 128.6 mm, vias 0 -> 9
- net com7: track 0.00 -> 121.9 mm, vias 0 -> 2
- net row1: track 0.00 -> 121.3 mm, vias 0 -> 9
- net row2: track 0.00 -> 120.8 mm, vias 0 -> 9
- net com6: track 0.00 -> 120.4 mm, vias 0 -> 2
- net com5: track 0.00 -> 119.3 mm, vias 0 -> 2
- net com4: track 0.00 -> 117.9 mm, vias 0 -> 2
- net row3: track 0.00 -> 117.3 mm, vias 0 -> 9
- net com3: track 0.00 -> 116.5 mm, vias 0 -> 2
- net row4: track 0.00 -> 116.4 mm, vias 0 -> 9
- net com2: track 0.00 -> 115.0 mm, vias 0 -> 2
- net row5: track 0.00 -> 113.8 mm, vias 0 -> 9
- net com1: track 0.00 -> 113.4 mm, vias 0 -> 2
- net com0: track 0.00 -> 112.0 mm, vias 0 -> 2
- net row6: track 0.00 -> 106.7 mm, vias 0 -> 9
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Other:
- board outline added: 100 x 40 mm

Commit message: e
Routing:
- net row10: track 30.4 -> 76.7 mm
Changed lines of the file:
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@@
 			(outputformat 1)
 			(mirror no)
-			(drillshape 1)
+			(drillshape 0)
 			(scaleselection 1)
 			(outputdirectory "")
@@
 	)
 	(segment
-		(start 179.7 110.128)
-		(end 180.128 110.128)
+		(start 143.801 122.676)
+		(end 143.125 122)
+		(width 0.2)
+		(layer "F.Cu")
+		(net 23)
+	)
+	(segment
+		(start 175.032521 122.676)
+		(end 143.801 122.676)
 		(width 0.2)
 		(layer "F.Cu")
@@
 	)
 	(segment
+		(start 179.7 110.128)
+		(end 179.7 118.008521)
+		(width 0.2)
+		(layer "F.Cu")
+		(net 23)
+	)
+	(segment
 		(start 143.1 119)
 		(end 141.975 119)
@@
 		(width 0.2)
 		(layer "F.Cu")
+		(net 23)
+	)
+	(segment
+		(start 179.7 118.008521)
+		(end 175.032521 122.676)
+		(width 0.2)
+		(layer "F.Cu")

Commit message: e
Parts:
- C1, C2: footprint Capacitor_SMD:C_0603_1608Metric_Pad1.08x0.95mm_HandSolder -> Capacitor_SMD:C_0805_2012Metric_Pad1.18x1.45mm_HandSolder
- D1, D10, D100, D101, D102, D103, D104, D105, D106, D107, D108, D109, D11, D110, D111, D112, D113, D114, D115, D116, D117, D118, D119, D12, D120, D121, D122, D123, D124, D125, D126, D127, D128, D13, D14, D15, D16, D17, D18, D19, D2, D20, D21, D22, D23, D24, D25, D26, D27, D28, D29, D3, D30, D31, D32, D33, D34, D35, D36, D37, D38, D39, D4, D40, D41, D42, D43, D44, D45, D46, D47, D48, D49, D5, D50, D51, D52, D53, D54, D55, D56, D57, D58, D59, D6, D60, D61, D62, D63, D64, D65, D66, D67, D68, D69, D7, D70, D71, D72, D73, D74, D75, D76, D77, D78, D79, D8, D80, D81, D82, D83, D84, D85, D86, D87, D88, D89, D9, D90, D91, D92, D93, D94, D95, D96, D97, D98, D99: footprint LED_SMD:LED_0603_1608Metric_Pad1.05x0.95mm_HandSolder -> LED_SMD:LED_0805_2012Metric_Pad1.15x1.40mm_HandSolder
- R1, R10, R2, R3, R4, R5, R6, R7, R8, R9: footprint Resistor_SMD:R_0603_1608Metric_Pad0.98x0.95mm_HandSolder -> Resistor_SMD:R_0805_2012Metric_Pad1.20x1.40mm_HandSolder
Connections:
- C1 pad 1: Net-(IC1-VDD) -> /-
- C1 pad 2: Net-(J1-Pin_1) -> /+
- C2 pad 1: Net-(J1-Pin_2) -> unconnected-(C2-Pad1)
- C2 pad 2: Net-(IC1-VSS) -> unconnected-(C2-Pad2)
- IC1 pad 1: Net-(IC1-VSS) -> /-
- IC1 pad 28: Net-(IC1-VDD) -> /+
- J1 pad 1: Net-(J1-Pin_1) -> /+
- J1 pad 2: Net-(J1-Pin_2) -> /-
Routing:
- net row0: track 128.6 -> 0.00 mm, vias 9 -> 0
- net com7: track 121.9 -> 0.00 mm, vias 2 -> 0
- net row1: track 121.3 -> 0.00 mm, vias 9 -> 0
- net row2: track 120.8 -> 0.00 mm, vias 9 -> 0
- net com6: track 120.4 -> 0.00 mm, vias 2 -> 0
- net com5: track 119.3 -> 0.00 mm, vias 2 -> 0
- net com4: track 117.9 -> 0.00 mm, vias 2 -> 0
- net row3: track 117.3 -> 0.00 mm, vias 9 -> 0
- net com3: track 116.5 -> 0.00 mm, vias 2 -> 0
- net row4: track 116.4 -> 0.00 mm, vias 9 -> 0
- net com2: track 115.0 -> 0.00 mm, vias 2 -> 0
- net row5: track 113.8 -> 0.00 mm, vias 9 -> 0
- net com1: track 113.4 -> 0.00 mm, vias 2 -> 0
- net com0: track 112.0 -> 0.00 mm, vias 2 -> 0
- net row6: track 106.7 -> 0.00 mm, vias 9 -> 0
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