File: led-pcb.kicad_sch (KiCad schematic)
At the start: 0 parts

Commit message: e
Parts:
- added D1, D10, D100, D11, D13, D15, D17, D20, D21, D23, D25, D27, D3, D30, D31, D33, D35, D37, D40, D41, D43, D45, D47, D5, D50, D51, D53, D55, D57, D60, D61, D63, D65, D67, D7, D70, D71, D73, D75, D77, D80, D81, D83, D85, D87, D90, D91, D93, D95, D97: LED, LED_SMD:LED_0603_1608Metric_Pad1.05x0.95mm_HandSolder, symbol Device:LED
- added D12, D14, D16, D18, D19, D2, D22, D24, D26, D28, D29, D32, D34, D36, D38, D39, D4, D42, D44, D46, D48, D49, D52, D54, D56, D58, D59, D6, D62, D64, D66, D68, D69, D72, D74, D76, D78, D79, D8, D82, D84, D86, D88, D89, D9, D92, D94, D96, D98, D99: LED, symbol Device:LED
- added U1: MAX7221xWG, Package_SO:SOIC-24W_7.5x15.4mm_P1.27mm, symbol Driver_LED:MAX7221xWG
Connections:
- new net: U1.4 (GND), U1.9 (GND)

Commit message: e
Parts:
- removed U1: MAX7221xWG, Package_SO:SOIC-24W_7.5x15.4mm_P1.27mm, symbol Driver_LED:MAX7221xWG
- added D101, D103, D105, D107, D109, D111, D113, D115, D117, D119, D121, D123, D125, D127: LED, LED_SMD:LED_0603_1608Metric_Pad1.05x0.95mm_HandSolder, symbol Device:LED
- added D102, D104, D106, D108, D110, D112, D114, D116, D118, D120, D122, D124, D126, D128: LED, symbol Device:LED
- added R1, R2, R3, R4, R5, R6, R7, R8: R_US, Resistor_SMD:R_0603_1608Metric, symbol Device:R_US
- D10, D100, D20, D30, D40, D50, D60, D70, D80, D90: footprint LED_SMD:LED_0603_1608Metric_Pad1.05x0.95mm_HandSolder -> (none)
- D19, D29, D39, D49, D59, D69, D79, D89, D9, D99: footprint (none) -> LED_SMD:LED_0603_1608Metric_Pad1.05x0.95mm_HandSolder
Connections:
- net at D49.1 (K): now also D50.1 (K), D51.1 (K), D52.1 (K), D53.1 (K), D54.1 (K), D55.1 (K), D56.1 (K)
- net at D49.2 (A): now also D1.2 (A), D17.2 (A), D25.2 (A), D33.2 (A), D41.2 (A), D57.2 (A), D65.2 (A), D73.2 (A), D81.2 (A), D89.2 (A), D9.2 (A), D97.2 (A), D105.2 (A), D113.2 (A), D121.2 (A), R1.2
- net at D23.1 (K): now also D17.1 (K), D18.1 (K), D19.1 (K), D20.1 (K), D21.1 (K), D22.1 (K), D24.1 (K)
- net at D23.2 (A): now also D15.2 (A), D31.2 (A), D39.2 (A), D47.2 (A), D55.2 (A), D63.2 (A), D7.2 (A), D71.2 (A), D79.2 (A), D87.2 (A), D95.2 (A), D103.2 (A), D111.2 (A), D119.2 (A), D127.2 (A), R7.2
- net at D16.1 (K): now also D10.1 (K), D11.1 (K), D12.1 (K), D13.1 (K), D14.1 (K), D15.1 (K), D9.1 (K)
- net at D16.2 (A): now also D24.2 (A), D32.2 (A), D40.2 (A), D48.2 (A), D56.2 (A), D64.2 (A), D72.2 (A), D8.2 (A), D80.2 (A), D88.2 (A), D96.2 (A), D104.2 (A), D112.2 (A), D120.2 (A), D128.2 (A), R8.2
- net at D100.1 (K): now also D97.1 (K), D98.1 (K), D99.1 (K), D101.1 (K), D102.1 (K), D103.1 (K), D104.1 (K)
- net at D100.2 (A): now also D12.2 (A), D20.2 (A), D28.2 (A), D36.2 (A), D4.2 (A), D44.2 (A), D52.2 (A), D60.2 (A), D68.2 (A), D76.2 (A), D84.2 (A), D92.2 (A), D108.2 (A), D116.2 (A), D124.2 (A), R4.2
- net at D37.1 (K): now also D33.1 (K), D34.1 (K), D35.1 (K), D36.1 (K), D38.1 (K), D39.1 (K), D40.1 (K)
- net at D37.2 (A): now also D13.2 (A), D21.2 (A), D29.2 (A), D45.2 (A), D5.2 (A), D53.2 (A), D61.2 (A), D69.2 (A), D77.2 (A), D85.2 (A), D93.2 (A), D101.2 (A), D109.2 (A), D117.2 (A), D125.2 (A), R5.2
- net at D50.2 (A): now also D10.2 (A), D18.2 (A), D2.2 (A), D26.2 (A), D34.2 (A), D42.2 (A), D58.2 (A), D66.2 (A), D74.2 (A), D82.2 (A), D90.2 (A), D98.2 (A), D106.2 (A), D114.2 (A), D122.2 (A), R2.2
- net at D35.2 (A): now also D11.2 (A), D19.2 (A), D27.2 (A), D3.2 (A), D43.2 (A), D51.2 (A), D59.2 (A), D67.2 (A), D75.2 (A), D91.2 (A), D99.2 (A), D107.2 (A), D115.2 (A), D123.2 (A), R3.2
- net at D43.1 (K): now also D41.1 (K), D42.1 (K), D44.1 (K), D45.1 (K), D46.1 (K), D47.1 (K), D48.1 (K)
- net at D6.1 (K): now also D1.1 (K), D2.1 (K), D3.1 (K), D4.1 (K), D5.1 (K), D7.1 (K), D8.1 (K)
- net at D6.2 (A): now also D14.2 (A), D22.2 (A), D30.2 (A), D38.2 (A), D46.2 (A), D54.2 (A), D62.2 (A), D70.2 (A), D78.2 (A), D86.2 (A), D94.2 (A), D102.2 (A), D110.2 (A), D118.2 (A), D126.2 (A), R6.2
- net at D81.1 (K): now also D82.1 (K), D83.1 (K), D84.1 (K), D85.1 (K), D86.1 (K), D87.1 (K), D88.1 (K)
- net at D63.1 (K): now also D57.1 (K), D58.1 (K), D59.1 (K), D60.1 (K), D61.1 (K), D62.1 (K), D64.1 (K)
- net at D94.1 (K): now also D89.1 (K), D90.1 (K), D91.1 (K), D92.1 (K), D93.1 (K), D95.1 (K), D96.1 (K)
- net at D75.1 (K): now also D73.1 (K), D74.1 (K), D76.1 (K), D77.1 (K), D78.1 (K), D79.1 (K), D80.1 (K)
- net at D25.1 (K): now also D26.1 (K), D27.1 (K), D28.1 (K), D29.1 (K), D30.1 (K), D31.1 (K), D32.1 (K)
- net at D67.1 (K): now also D65.1 (K), D66.1 (K), D68.1 (K), D69.1 (K), D70.1 (K), D71.1 (K), D72.1 (K)
- new net: D113.1 (K), D114.1 (K), D115.1 (K), D116.1 (K), D117.1 (K), D118.1 (K), D119.1 (K), D120.1 (K)
- new net: D121.1 (K), D122.1 (K), D123.1 (K), D124.1 (K), D125.1 (K), D126.1 (K), D127.1 (K), D128.1 (K)
- new net: D105.1 (K), D106.1 (K), D107.1 (K), D108.1 (K), D109.1 (K), D110.1 (K), D111.1 (K), D112.1 (K)

Commit message: e
Parts:
- added C1: C_Small_US 100nF, Capacitor_SMD:C_0603_1608Metric_Pad1.08x0.95mm_HandSolder, symbol Device:C_Small_US
- added C2: C_Small_US 1uF, Capacitor_SMD:C_0603_1608Metric_Pad1.08x0.95mm_HandSolder, symbol Device:C_Small_US
- added IC1: HT16K33A-28SSOP, HT16K33A-28SOP:SOP64P600X175-28N, symbol HT16K33A-28SOP:HT16K33A-28SSOP
- added J1: Conn_01x04_Pin, Connector_PinSocket_2.54mm:PinSocket_1x04_P2.54mm_Vertical, symbol Connector:Conn_01x04_Pin
- added R10, R9: R_US 4.7kΩ, Resistor_SMD:R_0603_1608Metric_Pad0.98x0.95mm_HandSolder, symbol Device:R_US
- D10, D100, D102, D104, D106, D108, D110, D112, D114, D116, D118, D12, D120, D122, D124, D126, D128, D14, D16, D18, D2, D20, D22, D24, D26, D28, D30, D32, D34, D36, D38, D4, D40, D42, D44, D46, D48, D50, D52, D54, D56, D58, D6, D60, D62, D64, D66, D68, D70, D72, D74, D76, D78, D8, D80, D82, D84, D86, D88, D90, D92, D94, D96, D98: footprint (none) -> LED_SMD:LED_0603_1608Metric_Pad1.05x0.95mm_HandSolder
- R1, R2, R3, R4, R5, R6, R7, R8: value R_US -> R_US 10Ω
Connections:
- net row14: now reaches D113.1 (K), D114.1 (K), D115.1 (K), D116.1 (K), D117.1 (K), D118.1 (K), D119.1 (K), D120.1 (K)
- net row14: now also IC1.11 (ROW14/K12)
- net col4: now reaches D101.2 (A), D109.2 (A), D117.2 (A), D125.2 (A), D13.2 (A), D21.2 (A), D29.2 (A), D37.2 (A), D45.2 (A), D5.2 (A), D53.2 (A), D61.2 (A), D69.2 (A), D77.2 (A), D85.2 (A), D93.2 (A), R5.2
- net row15: now reaches D121.1 (K), D122.1 (K), D123.1 (K), D124.1 (K), D125.1 (K), D126.1 (K), D127.1 (K), D128.1 (K)
- net row15: now also IC1.10 (ROW15/K13/INT)
- net col6: now reaches D103.2 (A), D111.2 (A), D119.2 (A), D127.2 (A), D15.2 (A), D23.2 (A), D31.2 (A), D39.2 (A), D47.2 (A), D55.2 (A), D63.2 (A), D7.2 (A), D71.2 (A), D79.2 (A), D87.2 (A), D95.2 (A), R7.2
- net row12: now reaches D100.1 (K), D101.1 (K), D102.1 (K), D103.1 (K), D104.1 (K), D97.1 (K), D98.1 (K), D99.1 (K)
- net row12: now also IC1.13 (ROW12/K10)
- net col0: now reaches D1.2 (A), D105.2 (A), D113.2 (A), D121.2 (A), D17.2 (A), D25.2 (A), D33.2 (A), D41.2 (A), D49.2 (A), D57.2 (A), D65.2 (A), D73.2 (A), D81.2 (A), D89.2 (A), D9.2 (A), D97.2 (A), R1.2
- net row5: now reaches D41.1 (K), D42.1 (K), D43.1 (K), D44.1 (K), D45.1 (K), D46.1 (K), D47.1 (K), D48.1 (K)
- net row5: now also IC1.20 (ROW5/K3)
- net row6: now reaches D49.1 (K), D50.1 (K), D51.1 (K), D52.1 (K), D53.1 (K), D54.1 (K), D55.1 (K), D56.1 (K)
- net row6: now also IC1.19 (ROW6/K4)
- net col2: now reaches D107.2 (A), D11.2 (A), D115.2 (A), D123.2 (A), D19.2 (A), D27.2 (A), D3.2 (A), D35.2 (A), D43.2 (A), D51.2 (A), D59.2 (A), D67.2 (A), D75.2 (A), D91.2 (A), D99.2 (A), R3.2
- net col2: now also D83.2 (A)
- net row1: now reaches D10.1 (K), D11.1 (K), D12.1 (K), D13.1 (K), D14.1 (K), D15.1 (K), D16.1 (K), D9.1 (K)
- net row1: now also IC1.24 (ROW1/A1)
- net row3: now reaches D25.1 (K), D26.1 (K), D27.1 (K), D28.1 (K), D29.1 (K), D30.1 (K), D31.1 (K), D32.1 (K)
- net row3: now also IC1.22 (ROW3/K1)
- net row11: now reaches D89.1 (K), D90.1 (K), D91.1 (K), D92.1 (K), D93.1 (K), D94.1 (K), D95.1 (K), D96.1 (K)
- net row11: now also IC1.14 (ROW11/K9)
- net row0: now reaches D1.1 (K), D2.1 (K), D3.1 (K), D4.1 (K), D5.1 (K), D6.1 (K), D7.1 (K), D8.1 (K)
- net row0: now also IC1.25 (ROW0/A2)
- net col5: now reaches D102.2 (A), D110.2 (A), D118.2 (A), D126.2 (A), D14.2 (A), D22.2 (A), D30.2 (A), D38.2 (A), D46.2 (A), D54.2 (A), D6.2 (A), D62.2 (A), D70.2 (A), D78.2 (A), D86.2 (A), D94.2 (A), R6.2
- net col7: now reaches D104.2 (A), D112.2 (A), D120.2 (A), D128.2 (A), D16.2 (A), D24.2 (A), D32.2 (A), D40.2 (A), D48.2 (A), D56.2 (A), D64.2 (A), D72.2 (A), D8.2 (A), D80.2 (A), D88.2 (A), D96.2 (A), R8.2
- net row4: now reaches D33.1 (K), D34.1 (K), D35.1 (K), D36.1 (K), D37.1 (K), D38.1 (K), D39.1 (K), D40.1 (K)
- net row4: now also IC1.21 (ROW4/K2)
- net col3: now reaches D100.2 (A), D108.2 (A), D116.2 (A), D12.2 (A), D124.2 (A), D20.2 (A), D28.2 (A), D36.2 (A), D4.2 (A), D44.2 (A), D52.2 (A), D60.2 (A), D68.2 (A), D76.2 (A), D84.2 (A), D92.2 (A), R4.2
- net row9: now reaches D73.1 (K), D74.1 (K), D75.1 (K), D76.1 (K), D77.1 (K), D78.1 (K), D79.1 (K), D80.1 (K)
- net row9: now also IC1.16 (ROW9/K7)
- net row13: now reaches D105.1 (K), D106.1 (K), D107.1 (K), D108.1 (K), D109.1 (K), D110.1 (K), D111.1 (K), D112.1 (K)
- net row13: now also IC1.12 (ROW13/K11)
- net row10: now reaches D81.1 (K), D82.1 (K), D83.1 (K), D84.1 (K), D85.1 (K), D86.1 (K), D87.1 (K), D88.1 (K)
- net row10: now also IC1.15 (ROW10/K8)
- net col1: now reaches D10.2 (A), D106.2 (A), D114.2 (A), D122.2 (A), D18.2 (A), D2.2 (A), D26.2 (A), D34.2 (A), D42.2 (A), D50.2 (A), D58.2 (A), D66.2 (A), D74.2 (A), D82.2 (A), D90.2 (A), D98.2 (A), R2.2
- net row2: now reaches D17.1 (K), D18.1 (K), D19.1 (K), D20.1 (K), D21.1 (K), D22.1 (K), D23.1 (K), D24.1 (K)
- net row2: now also IC1.23 (ROW2/A0)
- net row7: now reaches D57.1 (K), D58.1 (K), D59.1 (K), D60.1 (K), D61.1 (K), D62.1 (K), D63.1 (K), D64.1 (K)
- net row7: now also IC1.18 (ROW7/K5)
- net com7: now reaches R8.1
- net com7: now also IC1.9 (COM7)
- net com2: now reaches R3.1
- net com2: now also IC1.4 (COM2/KS1)
- net row8: now reaches D65.1 (K), D66.1 (K), D67.1 (K), D68.1 (K), D69.1 (K), D70.1 (K), D71.1 (K), D72.1 (K)
- net row8: now also IC1.17 (ROW8/K6)
- net com0: now reaches R1.1
- net com0: now also IC1.2 (COM0/AD)
- net com3: now reaches R4.1
- net com3: now also IC1.5 (COM3/KS2)
- net com1: now reaches R2.1
- net com1: now also IC1.3 (COM1/KS0)
- net com5: now reaches R6.1
- net com5: now also IC1.7 (COM5)
- net com4: now reaches R5.1
- net com4: now also IC1.6 (COM4)
- net com6: now reaches R7.1
- net com6: now also IC1.8 (COM6)
- new net: C2.1, IC1.1 (VSS)
- new net: C2.2, J1.2 (Pin_2)
- new net: C1.2, J1.1 (Pin_1)
- new net: J1.3 (Pin_3), R9.2
- new net: J1.4 (Pin_4), R10.2
- new net: C1.1, IC1.28 (VDD)
- new net: IC1.26 (SCL), R10.1
- new net: IC1.27 (SDA), R9.1
Other:
- moved on the sheet: D1, D10, D100, D101, D102, D103, D104, D105, D106, D107, D108, D109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

Commit message: e
Parts:
- R1, R2, R3, R4, R5, R6, R7, R8: footprint Resistor_SMD:R_0603_1608Metric -> Resistor_SMD:R_0603_1608Metric_Pad0.98x0.95mm_HandSolder
Connections:
- net at C2.1: now also J1.2 (Pin_2); no longer IC1.1 (VSS)
- net at C2.2: now also IC1.1 (VSS); no longer J1.2 (Pin_2)
Other:
- moved on the sheet: C2
Changed lines of the file:
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@@
 	(symbol
 		(lib_id "Device:C_Small_US")
-		(at 92.71 20.32 270)
+		(at 92.71 20.32 90)
+		(mirror x)
 		(unit 1)
 		(exclude_from_sim no)
@@
 		(on_board yes)
 		(dnp no)
-		(fields_autoplaced yes)
 		(property "Reference" "C2"
-			(at 92.583 13.97 90)
+			(at 92.837 13.97 90)
 			(effects
 				(font
@@
 		)
 		(property "Value" "C_Small_US 1uF"
-			(at 92.583 16.51 90)
+			(at 92.837 16.51 90)
 			(effects
 				(font
@@
 			)
 		)
-		(property "Footprint" "Resistor_SMD:R_0603_1608Metric"
+		(property "Footprint" "Resistor_SMD:R_0603_1608Metric_Pad0.98x0.95mm_HandSolder"
 			(at 94.234 162.814 90)
 			(effects
@@
 			)
 		)
-		(property "Footprint" "Resistor_SMD:R_0603_1608Metric"
+		(property "Footprint" "Resistor_SMD:R_0603_1608Metric_Pad0.98x0.95mm_HandSolder"
 			(at 94.234 137.414 90)
 			(effects
@@
 			)
 		)
-		(property "Footprint" "Resistor_SMD:R_0603_1608Metric"
+		(property "Footprint" "Resistor_SMD:R_0603_1608Metric_Pad0.98x0.95mm_HandSolder"
 			(at 94.234 127.254 90)
 			(effects
@@
 			)
 		)
-		(property "Footprint" "Resistor_SMD:R_0603_1608Metric"
+		(property "Footprint" "Resistor_SMD:R_0603_1608Metric_Pad0.98x0.95mm_HandSolder"
 			(at 94.234 142.494 90)
 			(effects
@@
 			)
 		)
-		(property "Footprint" "Resistor_SMD:R_0603_1608Metric"
+		(property "Footprint" "Resistor_SMD:R_0603_1608Metric_Pad0.98x0.95mm_HandSolder"
 			(at 94.234 132.334 90)
 			(effects
@@
 			)
 		)
-		(property "Footprint" "Resistor_SMD:R_0603_1608Metric"
+		(property "Footprint" "Resistor_SMD:R_0603_1608Metric_Pad0.98x0.95mm_HandSolder"
 			(at 94.234 152.654 90)
 			(effects
@@
 			)
 		)
-		(property "Footprint" "Resistor_SMD:R_0603_1608Metric"
+		(property "Footprint" "Resistor_SMD:R_0603_1608Metric_Pad0.98x0.95mm_HandSolder"
 			(at 94.234 147.574 90)
 			(effects
@@
 			)
 		)
-		(property "Footprint" "Resistor_SMD:R_0603_1608Metric"
+		(property "Footprint" "Resistor_SMD:R_0603_1608Metric_Pad0.98x0.95mm_HandSolder"
 			(at 94.234 157.734 90)
 			(effects

Commit message: e
Other:
- moved on the sheet: D1, D10, D100, D101, D102, D103, D104, D105, D106, D107, D108, D109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

Commit message: e
Connections:
- net at C2.1: no longer J1.2 (Pin_2)
- net at C2.2: no longer IC1.1 (VSS)
- net +: now reaches C1.2, J1.1 (Pin_1)
- net +: now also IC1.28 (VDD)
- net -: now reaches C1.1
- net -: now also IC1.1 (VSS), J1.2 (Pin_2); no longer IC1.28 (VDD)
Other:
- moved on the sheet: C1, C2, J1
Changed lines of the file:
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@@
 	)
 	(junction
+		(at 153.67 21.59)
+		(diameter 0)
+		(color 0 0 0 0)
+	)
+	(junction
 		(at 143.51 113.03)
 		(diameter 0)
@@
 	)
 	(junction
+		(at 153.67 16.51)
+		(diameter 0)
+		(color 0 0 0 0)
+	)
+	(junction
 		(at 120.65 102.87)
 		(diameter 0)
@@
 	(wire
 		(pts
-			(xy 148.59 25.4) (xy 157.48 25.4)
+			(xy 148.59 25.4) (xy 181.61 25.4)
 		)
 		(stroke
@@
 	(wire
 		(pts
-			(xy 157.48 19.05) (xy 146.05 19.05)
-		)
-		(stroke
-			(width 0)
-			(type default)
-		)
-	)
-	(wire
-		(pts
 			(xy 113.03 90.17) (xy 113.03 95.25)
 		)
@@
 	(wire
 		(pts
-			(xy 157.48 24.13) (xy 148.59 24.13)
+			(xy 181.61 24.13) (xy 148.59 24.13)
 		)
 		(stroke
@@
 	(wire
 		(pts
+			(xy 153.67 21.59) (xy 151.13 21.59)
+		)
+		(stroke
+			(width 0)
+			(type default)
+		)
+	)
+	(wire
+		(pts
 			(xy 177.8 87.63) (xy 177.8 90.17)
 		)
@@
 		)
 	)
+	(wire
+		(pts
+			(xy 151.13 21.59) (xy 151.13 11.43)
+		)
+		(stroke
+			(width 0)
+			(type default)
+		)
+	)
 	(bus
 		(pts
@@
 	(wire
 		(pts
-			(xy 90.17 12.7) (xy 90.17 20.32)
-		)
-		(stroke
-			(width 0)
-			(type default)
-		)
-	)
-	(wire
-		(pts
 			(xy 74.93 97.79) (xy 63.5 97.79)
 		)
@@
 	(wire
 		(pts
+			(xy 153.67 21.59) (xy 181.61 21.59)
+		)
+		(stroke
+			(width 0)
+			(type default)
+		)
+	)
+	(wire
+		(pts
 			(xy 63.5 123.19) (xy 63.5 125.73)
 		)
@@
 	(wire
 		(pts
+			(xy 140.97 16.51) (xy 140.97 20.32)
+		)
+		(stroke
+			(width 0)
+			(type default)
+		)
+	)
+	(wire
+		(pts
 			(xy 140.97 43.18) (xy 149.86 43.18)
 		)
@@
 	(wire
 		(pts
-			(xy 157.48 25.4) (xy 157.48 26.67)
+			(xy 181.61 25.4) (xy 181.61 26.67)
 		)
 		(stroke
@@
 	(wire
 		(pts
+			(xy 181.61 19.05) (xy 176.53 19.05)
+		)
+		(stroke
+			(width 0)
+			(type default)
+		)
+	)
+	(wire
+		(pts
 			(xy 63.5 113.03) (xy 74.93 113.03)
 		)
@@
 	(wire
 		(pts
+			(xy 151.13 11.43) (xy 95.25 11.43)
+		)
+		(stroke
+			(width 0)
+			(type default)
+		)
+	)
+	(wire
+		(pts
 			(xy 223.52 102.87) (xy 234.95 102.87)
 		)
@@
 	(wire
 		(pts
+			(xy 95.25 11.43) (xy 95.25 20.32)
+		)
+		(stroke
+			(width 0)
+			(type default)
+		)
+	)
+	(wire
+		(pts
 			(xy 97.79 107.95) (xy 97.79 110.49)
 		)
@@
 	(wire
 		(pts
+			(xy 176.53 19.05) (xy 176.53 16.51)
+		)
+		(stroke
+			(width 0)
+			(type default)
+		)
+	)
+	(wire
+		(pts
 			(xy 238.76 105.41) (xy 238.76 110.49)
 		)
@@
 	(wire
 		(pts
+			(xy 153.67 16.51) (xy 176.53 16.51)
+		)
+		(stroke
+			(width 0)
+			(type default)
+		)
+	)
+	(wire
+		(pts
 			(xy 193.04 110.49) (xy 193.04 115.57)
 		)
@@
 	(wire
 		(pts
-			(xy 152.4 21.59) (xy 152.4 12.7)
-		)
-		(stroke
-			(width 0)
-			(type default)
-		)
-	)
-	(wire
-		(pts
 			(xy 177.8 97.79) (xy 177.8 100.33)
 		)
@@
 	(wire
 		(pts
-			(xy 146.05 19.05) (xy 146.05 20.32)
-		)
-		(stroke
-			(width 0)
-			(type default)
-		)
-	)
-	(wire
-		(pts
 			(xy 166.37 113.03) (xy 166.37 115.57)
 		)
@@
 	(wire
 		(pts
-			(xy 90.17 12.7) (xy 152.4 12.7)
-		)
-		(stroke
-			(width 0)
-			(type default)
-		)
-	)
-	(wire
-		(pts
 			(xy 166.37 102.87) (xy 177.8 102.87)
 		)
@@
 	(wire
 		(pts
-			(xy 157.48 21.59) (xy 152.4 21.59)
+			(xy 223.52 123.19) (xy 234.95 123.19)
 		)
 		(stroke
@@
 	(wire
 		(pts
-			(xy 223.52 123.19) (xy 234.95 123.19)
+			(xy 140.97 16.51) (xy 153.67 16.51)
 		)
 		(stroke
@@
 		)
 	)
+	(label "-"
+		(at 179.07 21.59 0)
+		(effects
+			(font
+				(size 1.27 1.27)
+			)
+			(justify left bottom)
+		)
+	)
 	(label "col0"
 		(at 63.5 87.63 0)
@@
 		)
 	)
+	(label "+"
+		(at 179.07 19.05 0)
+		(effects
+			(font
+				(size 1.27 1.27)
+			)
+			(justify left bottom)
+		)
+	)
 	(global_label "com[0..7]"
 		(shape input)
@@
 	(symbol
 		(lib_id "Device:C_Small_US")
-		(at 92.71 20.32 90)
+		(at 68.58 50.8 0)
 		(mirror x)
 		(unit 1)
@@
 		(dnp no)
 		(property "Reference" "C2"
-			(at 92.837 13.97 90)
+			(at 62.23 50.673 90)
 			(effects
 				(font
@@
 		)
 		(property "Value" "C_Small_US 1uF"
-			(at 92.837 16.51 90)
+			(at 64.77 50.673 90)
 			(effects
 				(font
@@
 		)
 		(property "Footprint" "Capacitor_SMD:C_0603_1608Metric_Pad1.08x0.95mm_HandSolder"
-			(at 92.71 20.32 0)
+			(at 68.58 50.8 0)
 			(effects
 				(font
@@
 		)
 		(property "Datasheet" ""
-			(at 92.71 20.32 0)
+			(at 68.58 50.8 0)
 			(effects
 				(font
@@
 		)
 		(property "Description" "capacitor, small US symbol"
-			(at 92.71 20.32 0)
+			(at 68.58 50.8 0)
 			(effects
 				(font
@@
 	(symbol
 		(lib_id "Connector:Conn_01x04_Pin")
-		(at 162.56 21.59 0)
+		(at 186.69 21.59 0)
 		(mirror y)
 		(unit 1)
@@
 		(dnp no)
 		(property "Reference" "J1"
-			(at 161.925 13.97 0)
+			(at 186.055 13.97 0)
 			(effects
 				(font
@@
 		)
 		(property "Value" "Conn_01x04_Pin"
-			(at 161.925 16.51 0)
+			(at 186.055 16.51 0)
 			(effects
 				(font
@@
 		)
 		(property "Footprint" "Connector_PinSocket_2.54mm:PinSocket_1x04_P2.54mm_Vertical"
-			(at 162.56 21.59 0)
+			(at 186.69 21.59 0)
 			(effects
 				(font
@@
 		)
 		(property "Datasheet" "~"
-			(at 162.56 21.59 0)
+			(at 186.69 21.59 0)
 			(effects
 				(font
@@
 		)
 		(property "Description" "Generic connector, single row, 01x04, script generated"
-			(at 162.56 21.59 0)
+			(at 186.69 21.59 0)
 			(effects
 				(font
@@
 	(symbol
 		(lib_id "Device:C_Small_US")
-		(at 143.51 20.32 90)
+		(at 153.67 19.05 180)
 		(unit 1)
 		(exclude_from_sim no)
@@
 		(fields_autoplaced yes)
 		(property "Reference" "C1"
-			(at 143.637 13.97 90)
+			(at 156.21 17.6529 0)
 			(effects
 				(font
 					(size 1.27 1.27)
 				)
+				(justify right)
 			)
 		)
 		(property "Value" "C_Small_US 100nF"
-			(at 143.637 16.51 90)
+			(at 156.21 20.1929 0)
 			(effects
 				(font
 					(size 1.27 1.27)
 				)
+				(justify right)
 			)
 		)
 		(property "Footprint" "Capacitor_SMD:C_0603_1608Metric_Pad1.08x0.95mm_HandSolder"
-			(at 143.51 20.32 0)
+			(at 153.67 19.05 0)
 			(effects
 				(font
@@
 		)
 		(property "Datasheet" ""
-			(at 143.51 20.32 0)
+			(at 153.67 19.05 0)
 			(effects
 				(font
@@
 		)
 		(property "Description" "capacitor, small US symbol"
-			(at 143.51 20.32 0)
+			(at 153.67 19.05 0)
 			(effects
 				(font

Commit message: e
Parts:
- C1, C2: footprint Capacitor_SMD:C_0603_1608Metric_Pad1.08x0.95mm_HandSolder -> Capacitor_SMD:C_0805_2012Metric_Pad1.18x1.45mm_HandSolder
- D1, D10, D100, D101, D102, D103, D104, D105, D106, D107, D108, D109, D11, D110, D111, D112, D113, D114, D115, D116, D117, D118, D119, D12, D120, D121, D122, D123, D124, D125, D126, D127, D128, D13, D14, D15, D16, D17, D18, D19, D2, D20, D21, D22, D23, D24, D25, D26, D27, D28, D29, D3, D30, D31, D32, D33, D34, D35, D36, D37, D38, D39, D4, D40, D41, D42, D43, D44, D45, D46, D47, D48, D49, D5, D50, D51, D52, D53, D54, D55, D56, D57, D58, D59, D6, D60, D61, D62, D63, D64, D65, D66, D67, D68, D69, D7, D70, D71, D72, D73, D74, D75, D76, D77, D78, D79, D8, D80, D81, D82, D83, D84, D85, D86, D87, D88, D89, D9, D90, D91, D92, D93, D94, D95, D96, D97, D98, D99: footprint LED_SMD:LED_0603_1608Metric_Pad1.05x0.95mm_HandSolder -> LED_SMD:LED_0805_2012Metric_Pad1.15x1.40mm_HandSolder
- R1, R10, R2, R3, R4, R5, R6, R7, R8, R9: footprint Resistor_SMD:R_0603_1608Metric_Pad0.98x0.95mm_HandSolder -> Resistor_SMD:R_0805_2012Metric_Pad1.20x1.40mm_HandSolder
Other:
- moved on the sheet: C1
